File: CM4Carrier.kicad_pcb (KiCad board)
At the start: 4 copper layers, 100 x 100 mm, 33 parts, among them J101 Conn_02x10_Row_Letter_First, J102 Conn_01x03_Pin, J201 DF40C-100DS-0.4V_51_, J202 DF40C-100DS-0.4V_51_, J301 HR911130A, U201 SN74LV1T34DBV, U301 TPD4EUSB30, U302 TPD4EUSB30, U401 RT9742GGJ5

Commit message: chore: migrate <<HASH>> placeholder to <<VERSION>> (#6)
Aligns the KiCad title-block placeholder with the new versioning concept
documented at oe5xrx.org/docs/remote-station/hardware/versioning/.

The placeholder is substituted at CI time:
- Release build:  v1.5 → "1.5" (semver only, no `v`, no SHA)
- Debug build:    "BETA-<short-commit>"

No electrical or layout change — pure text replacement on the title-block
silkscreen text. Requires HW-Module-CI feat/version-placeholder
(OE5XRX/HW-Module-CI#4) to be merged first; otherwise CI substitutes
the old <<HASH>> token and leaves the new <<VERSION>> string literal
in the title block until the CI side catches up.

Co-authored-by: Claude Opus 4.7 <noreply@anthropic.com>
Other:
- board text added: "<<VERSION>>"
- board text removed: "<<HASH>>"
Changed lines of the file:
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@@
 	(title_block
 		(title "CM4")
-		(rev "<<HASH>>")
+		(rev "<<VERSION>>")
 		(company "Amateurfunkclub für Remote Stationen")
 		(comment 1 "JLC04161H-7628")
@@
 		)
 	)
-	(gr_text "<<HASH>>"
+	(gr_text "<<VERSION>>"
 		(at 118.114 132.408 0)
 		(layer "F.SilkS")
